Commit message: Fixed errors in camera info settings. rviz file updated.

File: catkin_ws/src/aruco_track/resources/quad.urdf (robot description, URDF)
Before this commit: robot quad, 1 links, 0 joints
Links:
- link drone: geometry visual mesh filename=package://aruco_track/resources/quad.stl scale=0.001 0.001 0.001
